Commit message: URDF - Mass and Inertia configurad

File: urdf/barista_robot_model.urdf (robot description, URDF)
Before this commit: robot barista_bot, 13 links, 12 joints
Links:
- link back_pitch_link: mass None -> 0.11; geometry collision sphere radius=0.0352; visual sphere radius=0.0352
- link back_roll_link: mass None -> 0.12; geometry collision cylinder length=0.0206 radius=0.0352; visual cylinder length=0.0206 radius=0.0352
- link back_yaw_link: mass None -> 0.12; geometry collision cylinder length=0.0206 radius=0.0352; visual cylinder length=0.0206 radius=0.0352
- link chassis: mass None -> 2.92; geometry collision cylinder length=0.155 radius=0.178; visual cylinder length=0.155 radius=0.178
- link cup_holder_tray: mass None -> 1.31; geometry collision cylinder length=0.090 radius=0.160; visual cylinder length=0.090 radius=0.160
- link front_pitch_link: mass None -> 0.11; geometry collision sphere radius=0.0352; visual sphere radius=0.0352
- link front_roll_link: mass None -> 0.12; geometry collision cylinder length=0.0206 radius=0.0352; visual cylinder length=0.0206 radius=0.0352
- link front_yaw_link: mass None -> 0.12; geometry collision cylinder length=0.0206 radius=0.0352; visual cylinder length=0.0206 radius=0.0352
- link left_wheel: mass None -> 0.12; geometry collision cylinder length=0.0206 radius=0.0352; visual cylinder length=0.0206 radius=0.0352
- link right_wheel: mass None -> 0.12; geometry collision cylinder length=0.0206 radius=0.0352; visual cylinder length=0.0206 radius=0.0352
- link standoff_rod_left: mass None -> 0.41; geometry collision cylinder length=0.220 radius=0.020; visual cylinder length=0.220 radius=0.020
- link standoff_rod_right: mass None -> 0.41; geometry collision cylinder length=0.220 radius=0.020; visual cylinder length=0.220 radius=0.020

Commit message: URDF - Add Laser Model and Plugins (Need to Fix Robot Movement)

File: urdf/barista_robot_model.urdf (robot description, URDF)
Before this commit: robot barista_bot, 13 links, 12 joints
Links:
- added link laser_scan_frame
- added link laser_scan_link, mass 0.01; collision box size=0.074986 0.074935 0.0408; visual mesh filename=package://barista_robot_description/meshes/rplidar.dae scale=1.0 1.0 1.0
Joints:
- added joint laser_scan_frame_joint: type fixed, parent laser_scan_link, child laser_scan_frame, origin xyz=0 0 0.03 rpy=0 0 0, axis 0 0 0
- added joint laser_scan_link_joint: type fixed, parent chassis, child laser_scan_link, origin xyz=0.0 0.0 0.0780 rpy=0 0 0

Commit message: URDF - Changed the Laser Dae

File: urdf/barista_robot_model.urdf (robot description, URDF)
Before this commit: robot barista_robot, 15 links, 14 joints
Links:
- link laser_scan_link: geometry collision box size=0.074986 0.074935 0.0408; visual mesh filename=package://barista_robot_description/meshes/hokuyo_urg_04lx.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 scale=1.0 1.0 1.0
