Commit message: Spawn in Gazebo Two Robots

File: xacro/barista_robot_model.urdf.xacro (robot description, xacro)
@@ -1,4 +1,6 @@
 <?xml version="1.0"?>
 <robot xmlns:xacro="http://www.ros.org/wiki/xacro" name="barista_robot">
+<!-- Robot Name -->
+<xacro:property name="robot_name" value="$(arg robot_name)"/>
 <!-- Main Body Dimensions-->
 <xacro:property name="body_length" value="0.155"/>
@@ -13,5 +15,4 @@
 <xacro:include filename="$(find barista_robot_description)/xacro/cup_holder_tray.xacro" />
 <!-- Include Rviz Colors Macro-->
-<xacro:include filename="$(find barista_robot_description)/xacro/rviz_colors.xacro" />
 <link name="base_link">
   </link>
@@ -332,4 +333,5 @@
     <plugin name="box_bot_joint_state" filename="libgazebo_ros_joint_state_publisher.so">
       <ros>
+          <namespace>/${robot_name}</namespace>
           <remapping>~/out:=joint_states</remapping>
       </ros>
@@ -348,4 +350,8 @@
   <gazebo>
     <plugin filename="libgazebo_ros_diff_drive.so" name="differential_drive_controller">
+      <ros>
+          <namespace>/${robot_name}</namespace>
+          <remapping>/cmd_vel:=cmd_vel</remapping>
+      </ros>
       <!-- wheels -->
       <left_joint>joint_left_wheel</left_joint>
@@ -408,5 +414,5 @@
                 <plugin name="laser" filename="libgazebo_ros_ray_sensor.so">
                 <ros>
-                    <namespace></namespace>
+                    <namespace>/${robot_name}</namespace>
                     <remapping>~/out:=scan</remapping>
                 </ros>

Commit message: Fixed the Movement of the Robots

File: xacro/barista_robot_model.urdf.xacro (robot description, xacro)
@@ -6,4 +6,8 @@
 <xacro:property name="body_length" value="0.155"/>
 <xacro:property name="body_radius" value="0.178"/>
+<!-- Caster Wheels Dimensions-->
+<xacro:property name="caster_length" value="0.001"/>
+<xacro:property name="caster_radius" value="0.0045000000000000005"/>
+<xacro:property name="caster_sphere" value="0.0352"/>
 <!-- Include Laser -->
 <xacro:property name="include_laser" value="true"/>
@@ -133,5 +137,5 @@
     <origin rpy="0 1.5707 1.5707" xyz="0 0 0"/>
         <geometry>
-            <cylinder length="0.0206" radius="0.0352"/>
+            <cylinder length="${caster_length}" radius="${caster_radius}"/>
         </geometry>
         <material name="blue"/>
@@ -144,5 +148,5 @@
     <collision>
         <geometry>
-            <cylinder length="0.0206" radius="0.0352"/>
+            <cylinder length="${caster_length}" radius="${caster_radius}"/>
         </geometry>
     </collision>
@@ -163,5 +167,5 @@
         <origin rpy="0 1.5707 1.5707" xyz="0 0 0"/>
         <geometry>
-            <cylinder length="0.0206" radius="0.0352"/>
+            <cylinder length="${caster_length}" radius="${caster_radius}"/>
         </geometry>
         <material name="red"/>
@@ -174,5 +178,5 @@
     <collision>
         <geometry>
-            <cylinder length="0.0206" radius="0.0352"/>
+            <cylinder length="${caster_length}" radius="${caster_radius}"/>
         </geometry>
     </collision>
@@ -193,5 +197,5 @@
         <origin rpy="0 1.5707 1.5707" xyz="0 0 0"/>
         <geometry>
-            <sphere radius="0.0352"/>
+            <sphere radius="${caster_sphere}"/>
         </geometry>
         <material name="green_dark"/>
@@ -228,5 +232,5 @@
         <origin rpy="0 1.5707 1.5707" xyz="0 0 0"/>
         <geometry>
-          <cylinder length="0.0206" radius="0.0352"/>
+          <cylinder length="${caster_length}" radius="${caster_radius}"/>
         </geometry>
         <material name="blue"/>
@@ -239,5 +243,5 @@
     <collision>
         <geometry>
-            <cylinder length="0.0206" radius="0.0352"/>
+            <cylinder length="${caster_length}" radius="${caster_radius}"/>
         </geometry>
         </collision>
@@ -258,5 +262,5 @@
         <origin rpy="0 1.5707 1.5707" xyz="0 0 0"/>
         <geometry>
-          <cylinder length="0.0206" radius="0.0352"/>
+          <cylinder length="${caster_length}" radius="${caster_radius}"/>
         </geometry>
         <material name="red"/>
@@ -269,5 +273,5 @@
     <collision>
         <geometry>
-            <cylinder length="0.0206" radius="0.0352"/>
+            <cylinder length="${caster_length}" radius="${caster_radius}"/>
         </geometry>
     </collision>
@@ -288,5 +292,5 @@
         <origin rpy="0 1.5707 1.5707" xyz="0 0 0"/>
         <geometry>
-            <sphere radius="0.0352"/>
+            <sphere radius="${caster_sphere}"/>
         </geometry>
         <material name="green_light"/>
@@ -345,4 +349,5 @@
       <joint_name>front_pitch_joint</joint_name>
       <joint_name>back_pitch_joint</joint_name>
+      <joint_name>base_link_joint</joint_name>
     </plugin>
   </gazebo>
